File: hardware/boards/breakout/Breakout.sch (EAGLE design)
At the start: 4 parts

Commit message: added master changes
Changed lines of the file:
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@@
 <?xml version="1.0" encoding="utf-8"?>
 <!DOCTYPE eagle SYSTEM "eagle.dtd">
-<eagle version="7.0.0">
+<eagle version="7.2.0">
 <drawing>
 <settings>
