File: hardware/boards/breakout/Breakout_v2.brd (EAGLE design)
At the start: 42 x 42 mm, 6 parts

Commit message: Finished breakout v2
Parts:
- moved U$2 30.2 mm to (21.7, 32.7)
Routing:
- net N$23: track 6.51 -> 0.00 mm
- net BATV_BUS: track 23.9 -> 30.4 mm
- net +3V3_BUS: track 14.6 -> 18.5 mm
- net N$26: track 3.65 -> 0.00 mm
- net +3V3_SW1: track 8.97 -> 8.95 mm, vias 1 -> 0
- net BATV_SW1: track 9.50 -> 9.49 mm, vias 1 -> 0
- net +3V3_SW2: vias 1 -> 0
- net BATV_SW2: vias 1 -> 0
